Commit message: Update digital twin to round EE

File: ws/src/tendon_driven_finger/urdf/tendon_driven_finger.urdf (robot description, URDF)
Before this commit: robot tendon_driven_finger, 6 links, 5 joints
Links:
- link top: geometry collision box size=${width} ${length} 0.057; visual mesh filename=package://tendon_driven_finger/meshes/round-top.STL scale=0.001 0.001 0.001

Commit message: Add wrench visualization at the ee

File: ws/src/tendon_driven_finger/urdf/tendon_driven_finger.urdf (robot description, URDF)
Before this commit: robot tendon_driven_finger, 6 links, 5 joints
Links:
- added link ee
Joints:
- added joint ee_connector: type fixed, parent top, child ee, origin xyz=0.0 0.0 ${-(1.15*joint_offset)} rpy=${pi} 0 0

Commit message: Add Drone visualization to rviz

File: ws/src/tendon_driven_finger/urdf/tendon_driven_finger.urdf (robot description, URDF)
Before this commit: robot tendon_driven_finger, 7 links, 6 joints
Links:
- removed link world_connector
- added link world
Joints:
- joint world_joint: parent world_connector -> world
