Commit message: Rename Package to 'am_vis'

File: ws/src/am_vis/urdf/am.urdf (robot description, URDF)
Before this commit: robot am, 8 links, 7 joints
Links:
- link arm_base: geometry collision box size=0.08 0.05 0.05; visual mesh filename=package://am_vis/meshes/SensorizedBase.STL scale=0.001 0.001 0.001
- link base: geometry collision box size=0.5 0.5 0.25; visual mesh filename=package://am_vis/meshes/Holybro-X500-V2.STL scale=0.001 0.001 0.001
- link bottom: geometry collision box size=${width} ${length} 0.07; visual mesh filename=package://am_vis/meshes/SensorizedBottom.STL scale=0.001 0.001 0.001
- link middle: geometry collision box size=${width} ${length} 0.07; visual mesh filename=package://am_vis/meshes/SensorizedMiddle.STL scale=0.001 0.001 0.001
- link top: geometry collision box size=${width} ${length} 0.057; visual mesh filename=package://am_vis/meshes/round-top.STL scale=0.001 0.001 0.001

File: ws/src/am_vis/urdf/tendon_driven_finger.urdf (robot description, URDF)
Before this commit: robot tendon_driven_finger, 7 links, 6 joints
Links:
- link base: geometry collision box size=0.08 0.05 0.05; visual mesh filename=package://am_vis/meshes/SensorizedBase.STL scale=0.001 0.001 0.001
- link bottom: geometry collision box size=${width} ${length} 0.07; visual mesh filename=package://am_vis/meshes/SensorizedBottom.STL scale=0.001 0.001 0.001
- link middle: geometry collision box size=${width} ${length} 0.07; visual mesh filename=package://am_vis/meshes/SensorizedMiddle.STL scale=0.001 0.001 0.001
- link top: geometry collision box size=${width} ${length} 0.057; visual mesh filename=package://am_vis/meshes/round-top.STL scale=0.001 0.001 0.001

Commit message: Listen to px4 for pose; fix alignement of joint axes

File: ws/src/am_vis/urdf/am.urdf (robot description, URDF)
Before this commit: robot am, 8 links, 7 joints
Joints:
- joint arm_connector: origin xyz=0.27875 0.0 -0.018 rpy=0 0 0 -> xyz=0.27875 0.0 -0.018 rpy=0 ${pi} 0
- joint base_joint_pitch: origin xyz=0.0 0.0 ${-(joint_offset)} rpy=0 0 0 -> xyz=0.0 0.0 0.0315 rpy=0 0 0
- joint base_joint_roll: axis 0 1 0 -> 1 0 0; origin xyz=0.0 0.0 0.0 rpy=0 0 0 -> xyz=0.0 0.0 0.0 rpy=0 0 ${pi2}
- joint ee_connector: origin xyz=0.0 0.0 ${-(1.15*joint_offset)} rpy=${pi} 0 0 -> xyz=0.0 0.0 ${(1.05*joint_offset)} rpy=0 0 ${-pi2}
- joint middle_joint: axis 0 1 0 -> 1 0 0; origin xyz=0.0 0.0 ${-1.75*joint_offset} rpy=0 0 0 -> xyz=0.0 0.0 ${1.5*joint_offset} rpy=0 0 ${pi}
- joint top_joint: axis 0 1 0 -> 1 0 0; origin xyz=0.0 0.0 ${-(1.5*joint_offset)} rpy=0 0 0 -> xyz=0.0 0.0 ${(1.3*joint_offset)} rpy=0 0 ${-pi}

Commit message: Update drone mesh

File: ws/src/am_vis/urdf/am.urdf (robot description, URDF)
Before this commit: robot am, 8 links, 7 joints
Links:
- link base: geometry collision box size=0.5 0.5 0.25; visual mesh filename=package://am_vis/meshes/HolybroX500V2-withOBC.STL scale=0.001 0.001 0.001

Commit message: The arm is pointing in body y axis now

File: ws/src/am_vis/urdf/am.urdf (robot description, URDF)
Before this commit: robot am, 8 links, 7 joints
Joints:
- joint arm_connector: origin xyz=0.27875 0.0 -0.018 rpy=0 ${pi} 0 -> xyz=0.0 0.27875 -0.018 rpy=0 ${pi} ${pi2}

Commit message: Make urdf model use the colorful dae meshes

File: ws/src/am_vis/urdf/am.urdf (robot description, URDF)
Before this commit: robot am, 8 links, 7 joints
Links:
- link arm_base: geometry collision box size=0.08 0.05 0.05; visual mesh filename=package://am_vis/meshes/SensorizedBase.dae scale=1 1 1
- link base: geometry collision box size=0.5 0.5 0.25; visual mesh filename=package://am_vis/meshes/HolybroX500V2-withOBC.dae scale=1 1 1
- link bottom: geometry collision box size=${width} ${length} 0.07; visual mesh filename=package://am_vis/meshes/SensorizedBottom.dae scale=1 1 1
- link middle: geometry collision box size=${width} ${length} 0.07; visual mesh filename=package://am_vis/meshes/SensorizedMiddle.dae scale=1 1 1
- link top: geometry collision box size=${width} ${length} 0.057; visual mesh filename=package://am_vis/meshes/round-top.dae scale=1 1 1
Joints:
- joint arm_connector: origin xyz=0.0 0.27875 -0.018 rpy=0 ${pi} ${pi2} -> xyz=0.0 0.235 -0.018 rpy=0 ${pi} ${pi2}
